File: hardware/gx01-adapter-v2/gx01-adapter-v2-4layer.kicad_pcb (KiCad board)
At the start: 2 copper layers, 65 x 56.5 mm, 26 parts, among them J1 Pi GPIO 40-pin, J2 LCD 2x10 IDC, J3 Fan 1, J4 Fan 2, J5 FPB cable, Q1 AO3400A, U1 RV-3028-C7, U2 BME280, U3 MCP9808, U4 24LC32

Commit message: feat(hardware): GX-01 v2 HAT — placement iteration v2b routes successfully
State-of-technology test continuation. Two experiments added:

Option C (4-layer respin of v2 placement):
  - hardware/gx01-adapter-v2/gx01-adapter-v2-4layer.kicad_pcb
  - autoroute_4layer.py runs same placement with SetCopperLayerCount(4)
  - Result: still oscillated at 5-7 unrouted after 40 passes
  - Finding: adding layers ALONE does NOT fix a placement-driven routing
    problem. All 4 layers declared as signal in DSN; FreeRouting still
    couldn't escape local minimum.

Option B (2-layer placement iteration — v2b):
  - hardware/gx01-adapter-v2/layout_v2b.py — reworked placement that:
    * Removes I²C1 pull-ups from the J1↔J2 corridor
    * Splits RTC cluster (right side) vs EEPROM/sensor cluster (left)
    * Opens center of board for LCD signal routing
  - autoroute_v2b.py: CONVERGED. 444 tracks placed, clean SES produced.
  - DRC: 28 violations + 7 unconnected — all are PLACEMENT deltas
    (C4/C5 bypass caps overlap U3/U4 pads; C1/C2 courtyard overlap).
    Routing succeeded; only bypass-cap offsets need fixing.

Key state-of-tech finding: FreeRouting + scripted placement CAN produce
a fully-routed GX-01 v2 HAT at 36 nets on 2 layers. The v2-original
non-convergence was a placement problem, not a complexity limit.
Throwing 4 layers at it was unnecessary.

Next iteration to reach fab-ready (if pursued): move C4 +1mm from U3,
C5 +1mm from U4, C2 +2mm from C1. Rerun layout + autoroute. DRC should
then be clean or near-clean.

Co-Authored-By: Claude Opus 4.7 (1M context) <noreply@anthropic.com>
Other:
- copper layers 2 -> 4
